File: PowerBrigand-PCB/PowerBrigand.kicad_pcb (KiCad board)
At the start: 2 copper layers, 90 x 100 mm, 50 parts, among them J1 64Pin Edge Card, J2 Binding Post, J3 Binding Post, J4 Binding Post, J5 Anderson, J6 Anderson, J7 Anderson, Q1 2N3904, Q2 2N3904, SW1 On/Off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

Commit message: update license
Parts:
- added REF**: Symbol_CC-Noncommercial_SilkTop_Small, _NTSFootprints:Symbol_CC-Noncommercial_SilkTop_Small, B.Cu at (175.8, 94.4)
- moved REF** 12.2 mm to (175.8, 100.4)
- moved REF** 11.8 mm to (175.8, 82.7)
- moved REF** 6.25 mm to (175.8, 88.4)
Other:
- board text added: "Power Brigand (c)2020 Nathan Schenk"
Changed lines of the file:
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@@
   (general
     (thickness 1.6)
-    (drawings 13)
+    (drawings 14)
     (tracks 297)
     (zones 0)
-    (modules 50)
+    (modules 51)
     (nets 55)
   )
@@
   (title_block
     (title "PowerBrigand PCB")
-    (date 2020-07-12)
+    (date 2020-08-08)
     (rev 1.2)
     (company "N. Schenk")
+    (comment 1 "(c) 2020")
+    (comment 2 cc-by-nc-sa)
   )
   (layers
-    (0 F.Cu signal hide)
-    (31 B.Cu signal hide)
+    (0 F.Cu signal)
+    (31 B.Cu signal)
     (32 B.Adhes user hide)
     (33 F.Adhes user hide)
@@
     (36 B.SilkS user)
     (37 F.SilkS user)
-    (38 B.Mask user hide)
-    (39 F.Mask user)
+    (38 B.Mask user)
+    (39 F.Mask user hide)
     (40 Dwgs.User user)
     (41 Cmts.User user)
@@
     (add_net lcdRS)
   )
+  (module _NTSFootprints:Symbol_CC-Noncommercial_SilkTop_Small (layer B.Cu)
+    (at 175.764 94.41)
+    (descr "Symbol, CC-Noncommercial Alike, Silk Top Top, Small,")
+    (tags "Symbol, CC-Noncommercial Alike, Silk Top, Small,")
+    (attr virtual)
+    (fp_text reference REF** (at 0.59944 7.29996) (layer B.SilkS) hide
+      (effects (font (size 1 1) (thickness 0.15)) (justify mirror))
+    )
+    (fp_text value Symbol_CC-Noncommercial_SilkTop_Small (at 0.59944 -8.001) (layer B.Fab) hide
+      (effects (font (size 1 1) (thickness 0.15)) (justify mirror))
+    )
+    (fp_line (start 0.59944 2.4003) (end 0 2.49936) (layer B.SilkS) (width 0.381))
+    (fp_line (start 1.00076 2.30124) (end 0.59944 2.4003) (layer B.SilkS) (width 0.381))
+    (fp_line (start 1.50114 1.99898) (end 1.00076 2.30124) (layer B.SilkS) (width 0.381))
+    (fp_line (start 1.99898 1.50114) (end 1.50114 1.99898) (layer B.SilkS) (width 0.381))
+    (fp_line (start 2.30124 1.00076) (end 1.99898 1.50114) (layer B.SilkS) (width 0.381))
+    (fp_line (start 2.49936 0.39878) (end 2.30124 1.00076) (layer B.SilkS) (width 0.381))
+    (fp_line (start 2.49936 -0.20066) (end 2.49936 0.39878) (layer B.SilkS) (width 0.381))
+    (fp_line (start 2.4003 -0.8001) (end 2.49936 -0.20066) (layer B.SilkS) (width 0.381))
+    (fp_line (start 1.99898 -1.50114) (end 2.4003 -0.8001) (layer B.SilkS) (width 0.381))
+    (fp_line (start 1.50114 -1.99898) (end 1.99898 -1.50114) (layer B.SilkS) (width 0.381))
+    (fp_line (start 0.89916 -2.30124) (end 1.50114 -1.99898) (layer B.SilkS) (width 0.381))
+    (fp_line (start 0.29972 -2.49936) (end 0.89916 -2.30124) (layer B.SilkS) (width 0.381))
+    (fp_line (start -0.50038 -2.49936) (end 0.29972 -2.49936) (layer B.SilkS) (width 0.381))
+    (fp_line (start -1.19888 -2.19964) (end -0.50038 -2.49936) (layer B.SilkS) (width 0.381))
+    (fp_line (start -1.69926 -1.80086) (end -1.19888 -2.19964) (layer B.SilkS) (width 0.381))
+    (fp_line (start -2.30124 -1.09982) (end -1.69926 -1.80086) (layer B.SilkS) (width 0.381))
+    (fp_line (start -2.49936 -0.29972) (end -2.30124 -1.09982) (layer B.SilkS) (width 0.381))
+    (fp_line (start -2.49936 0.29972) (end -2.49936 -0.29972) (layer B.SilkS) (width 0.381))
+    (fp_line (start -2.4003 0.8001) (end -2.49936 0.29972) (layer B.SilkS) (width 0.381))
+    (fp_line (start -2.19964 1.19888) (end -2.4003 0.8001) (layer B.SilkS) (width 0.381))
+    (fp_line (start -1.69926 1.80086) (end -2.19964 1.19888) (layer B.SilkS) (width 0.381))
+    (fp_line (start -1.19888 2.19964) (end -1.69926 1.80086) (layer B.SilkS) (width 0.381))
+    (fp_line (start -0.70104 2.4003) (end -1.19888 2.19964) (layer B.SilkS) (width 0.381))
+    (fp_line (start -0.09906 2.49936) (end -0.70104 2.4003) (layer B.SilkS) (width 0.381))
+    (fp_line (start 0 2.49936) (end -0.09906 2.49936) (layer B.SilkS) (width 0.381))
+    (fp_line (start 0.70104 1.00076) (end 0.89916 1.19888) (layer B.SilkS) (width 0.381))
+    (fp_line (start 0.39878 1.09982) (end 0.70104 1.00076) (layer B.SilkS) (width 0.381))
+    (fp_line (start 0.09906 1.19888) (end 0.39878 1.09982) (layer B.SilkS) (width 0.381))
+    (fp_line (start -0.29972 1.09982) (end 0.09906 1.19888) (layer B.SilkS) (width 0.381))
+    (fp_line (start -0.50038 0.89916) (end -0.29972 1.09982) (layer B.SilkS) (width 0.381))
+    (fp_line (start -0.59944 0.70104) (end -0.50038 0.89916) (layer B.SilkS) (width 0.381))
+    (fp_line (start -0.50038 0.39878) (end -0.59944 0.70104) (layer B.SilkS) (width 0.381))
+    (fp_line (start -0.29972 0.20066) (end -0.50038 0.39878) (layer B.SilkS) (width 0.381))
+    (fp_line (start 0.29972 0.09906) (end -0.29972 0.20066) (layer B.SilkS) (width 0.381))
+    (fp_line (start 0.70104 -0.20066) (end 0.29972 0.09906) (layer B.SilkS) (width 0.381))
+    (fp_line (start 0.8001 -0.50038) (end 0.70104 -0.20066) (layer B.SilkS) (width 0.381))
+    (fp_line (start 0.8001 -0.8001) (end 0.8001 -0.50038) (layer B.SilkS) (width 0.381))
+    (fp_line (start 0.70104 -1.00076) (end 0.8001 -0.8001) (layer B.SilkS) (width 0.381))
+    (fp_line (start 0.50038 -1.19888) (end 0.70104 -1.00076) (layer B.SilkS) (width 0.381))
+    (fp_line (start 0.20066 -1.30048) (end 0.50038 -1.19888) (layer B.SilkS) (width 0.381))
+    (fp_line (start -0.50038 -1.30048) (end 0.20066 -1.30048) (layer B.SilkS) (width 0.381))
+    (fp_line (start -0.8001 -1.19888) (end -0.50038 -1.30048) (layer B.SilkS) (width 0.381))
+    (fp_line (start -0.8001 -1.00076) (end -0.8001 -1.19888) (layer B.SilkS) (width 0.381))
+    (fp_line (start -0.70104 -1.00076) (end -0.8001 -1.00076) (layer B.SilkS) (width 0.381))
+    (fp_line (start -0.20066 -1.09982) (end -0.70104 -1.00076) (layer B.SilkS) (width 0.381))
+    (fp_line (start 0.29972 -1.00076) (end -0.20066 -1.09982) (layer B.SilkS) (width 0.381))
+    (fp_line (start 0.59944 -0.8001) (end 0.29972 -1.00076) (layer B.SilkS) (width 0.381))
+    (fp_line (start 0.59944 -0.39878) (end 0.59944 -0.8001) (layer B.SilkS) (width 0.381))
+    (fp_line (start 0.29972 -0.20066) (end 0.59944 -0.39878) (layer B.SilkS) (width 0.381))
+    (fp_line (start -0.50038 0.09906) (end 0.29972 -0.20066) (layer B.SilkS) (width 0.381))
+    (fp_line (start -0.70104 0.29972) (end -0.50038 0.09906) (layer B.SilkS) (width 0.381))
+    (fp_line (start -0.8001 0.59944) (end -0.70104 0.29972) (layer B.SilkS) (width 0.381))
+    (fp_line (start -0.8001 0.89916) (end -0.8001 0.59944) (layer B.SilkS) (width 0.381))
+    (fp_line (start -0.70104 1.09982) (end -0.8001 0.89916) (layer B.SilkS) (width 0.381))
+    (fp_line (start -0.50038 1.30048) (end -0.70104 1.09982) (layer B.SilkS) (width 0.381))
+    (fp_line (start -0.29972 1.39954) (end -0.50038 1.30048) (layer B.SilkS) (width 0.381))
+    (fp_line (start 0.39878 1.39954) (end -0.29972 1.39954) (layer B.SilkS) (width 0.381))
+    (fp_line (start 0.8001 1.30048) (end 0.39878 1.39954) (layer B.SilkS) (width 0.381))
+    (fp_line (start 0.89916 1.19888) (end 0.8001 1.30048) (layer B.SilkS) (width 0.381))
+    (fp_line (start -2.30124 0.89916) (end 2.4003 -0.8001) (layer B.SilkS) (width 0.381))
+    (fp_line (start -2.4003 0.8001) (end 2.19964 -0.89916) (layer B.SilkS) (width 0.381))
+    (fp_line (start 0 1.50114) (end 0 1.80086) (layer B.SilkS) (width 0.381))
+    (fp_line (start 0 -1.80086) (end 0 -1.69926) (layer B.SilkS) (width 0.381))
+    (fp_line (start 0 -1.30048) (end 0 -1.80086) (layer B.SilkS) (width 0.381))
+  )
   (module MountingHole:MountingHole_3.2mm_M3_Pad (layer F.Cu)
     (at 119.764 115.66)
@@
   )
   (module _NTSFootprints:Symbol_CreativeCommons_CopperTop_Type2_Small (layer B.Cu)
-    (at 176.014 94.41 180)
+    (at 175.764 82.66 180)
     (descr "Symbol, Creative Commons, CopperTop, Type 2, Small,")
     (tags "Symbol, Creative Commons, CopperTop, Type 2, Small,")
@@
   )
   (module _NTSFootprints:Symbol_CC-ShareAlike_SilkTop_Small (layer B.Cu)
-    (at 175.764 88.16 180)
+    (at 175.764 100.41 180)
     (descr "Symbol, CC-Share Alike, Copper Top, Small,")
     (tags "Symbol, CC-Share Alike, Copper Top, Small,")
@@
   )
   (module _NTSFootprints:Symbol_CC-Attribution_SilkTop_Small (layer B.Cu)
-    (at 175.764 82.16 180)
+    (at 175.764 88.41 180)
     (descr "Symbol, CC-Share Alike, Copper Top, Small,")
     (tags "Symbol, CC-Share Alike, Copper Top, Small,")
@@
       (net 32 GNDPWR))
   )
+  (gr_text "Power Brigand (c)2020 Nathan Schenk" (at 145.264 58.66) (layer B.SilkS)
+    (effects (font (size 1 1) (thickness 0.15)) (justify mirror))
+  )
   (gr_text schenktronics.com (at 101.764 49.66 90) (layer F.SilkS)
